File: kicad/penmouse without charger.kicad_pcb (KiCad board)
At the start: 2 copper layers, 15.1 x 83.6 mm, 20 parts, among them J1 Conn_01x04_Socket, J2 Conn_01x04_Socket, SW1 SW_Push, SW2 SW_Push, SW3 SW_Push, U1 ATmega328P-P, U3 TPS61023DRLT, Y2 Crystal

Commit message: kicad files
Parts:
- C4, C5: footprint Capacitor_SMD:C_0402_1005Metric -> Capacitor_SMD:C_0603_1608Metric
- L3: footprint Inductor_SMD:L_0402_1005Metric -> Inductor_SMD:L_0201_0603Metric
- moved C5 1.10 mm to (116.9, 68.0)
Routing:
- net GND: track 142.0 -> 143.5 mm
- net vcc2: track 60.1 -> 59.4 mm
- net Net-(C4-Pad2): track 1.04 -> 1.57 mm
